Commit message: change urdf tag for gazebo7

File: mrsl_quadrotor_description/urdf/dragon_ddk/rgbd_camera.urdf.xacro (robot description, xacro)
@@ -17,7 +17,5 @@
           <origin xyz="0 0 0" rpy="0 0 0" />
           <geometry>
-            <box>
-              <size>0.001 0.001 0.001</size>
-            </box>
+              <box size="0.001 0.001 0.001" />
           </geometry>
         </visual>
@@ -25,7 +23,5 @@
           <origin xyz="0 0 0" rpy="0 0 0" />
           <geometry>
-            <box>
-              <size>0.001 0.001 0.001</size>
-            </box>
+            <box size="0.001 0.001 0.001" />
           </geometry>
         </collision>
