Commit message: Fix vio,  clean simulation

File: mrsl_quadrotor_description/urdf/dragon_ddk/dragon_ddk_so3.urdf.xacro (robot description, xacro)
@@ -20,7 +20,7 @@
       </visual>
       <collision>
-        <origin xyz="0 0 0" rpy="0 0 0" />
+        <origin xyz="0 0 -0.05" rpy="0 0 0" />
         <geometry>
-          <cylinder radius="0.15" length="0.1"/>
+          <cylinder radius="0.15" length="0.15"/>
         </geometry>
       </collision>
@@ -167,7 +167,7 @@
       <plugin filename="libgazebo_ros_imu_sensor.so" name="imu_plugin">
         <topicName>imu</topicName>
-        <bodyName>imu</bodyName>
+        <bodyName>imu_joint</bodyName>
         <updateRateHZ>100.0</updateRateHZ>
-        <gaussianNoise>0.0</gaussianNoise>
+        <gaussianNoise>0.000</gaussianNoise>
         <xyzOffset>0 0 0</xyzOffset>
         <rpyOffset>0 0 0</rpyOffset>

File: mrsl_quadrotor_description/urdf/dragon_ddk/stereo_camera.urdf.xacro (robot description, xacro)
@@ -8,5 +8,5 @@
   <xacro:property name="frame_id" value="camera" />
   <xacro:property name="focal_length" value="320" />
-  <xacro:property name="hack_baseline" value="0.10" />
+  <xacro:property name="hack_baseline" value="0.08" />
   <xacro:property name="frame_rate" value="15" />
   <xacro:macro name="stereo_camera" params="name parent *origin">
@@ -34,5 +34,5 @@
         <update_rate>${frame_rate}</update_rate>
         <camera name="left">
-          <pose>0 ${hack_baseline} 0 0 0 0</pose>
+          <pose>0 0 0 0 0 0</pose>
           <horizontal_fov>${hfov}</horizontal_fov>
           <image>
@@ -66,5 +66,5 @@
           <cameraInfoTopicName>camera_info</cameraInfoTopicName>
           <frameName>${frame_id}</frameName>
-          <hackBaseline>${2 * hack_baseline}</hackBaseline>
+          <hackBaseline>${hack_baseline}</hackBaseline>
           <CxPrime>${(image_width+1)/2}</CxPrime>
           <Cx>${(image_width+1)/2}</Cx>
