Commit message: fix downward camera rotation (was pointing at itself). increase publish rates of cameras

File: mrsl_quadrotor_description/urdf/dragon_ddk/camera.urdf.xacro (robot description, xacro)
@@ -24,5 +24,5 @@
     <gazebo reference="${name}_link">
       <sensor type="camera" name="${name}">
-        <update_rate>5.0</update_rate>
+        <update_rate>100.0</update_rate>
         <camera name="head">
           <horizontal_fov>${M_PI/2}</horizontal_fov>

File: mrsl_quadrotor_description/urdf/dragon_ddk/dragon_ddk_so3.urdf.xacro (robot description, xacro)
@@ -164,23 +164,4 @@
      </gazebo>
 <!--IMU Plugin-->
-  <gazebo reference="imu">
-    <gravity>true</gravity>
-    <sensor name="imu_sensor" type="imu">
-      <always_on>true</always_on>
-      <update_rate>100</update_rate>
-      <visualize>true</visualize>
-      <topic>__default_topic__</topic>
-      <plugin filename="libgazebo_ros_imu_sensor.so" name="imu_plugin">
-        <topicName>imu</topicName>
-        <bodyName>imu_joint</bodyName>
-        <updateRateHZ>100.0</updateRateHZ>
-        <gaussianNoise>0.000</gaussianNoise>
-        <xyzOffset>0 0 0</xyzOffset>
-        <rpyOffset>0 0 0</rpyOffset>
-        <frameName>imu</frameName>
-      </plugin>
-      <pose>0 0 0 0 0 0</pose>
-    </sensor>
-  </gazebo>
   </xacro:macro>
   <xacro:quadrotor_base_macro/>

File: mrsl_quadrotor_description/urdf/dragon_ddk/sensors.urdf.xacro (robot description, xacro)
@@ -3,5 +3,5 @@
   <xacro:include filename="$(find mrsl_quadrotor_description)/urdf/dragon_ddk/camera.urdf.xacro" />
   <xacro:monocular_camera name="dfc_camera" parent="dfc">
-    <origin xyz="0.0 0.0 0.0" rpy="${M_PI} ${M_PI/2} -${M_PI/2}"/>
+    <origin xyz="0.0 0.0 0.0" rpy="${M_PI} -${M_PI/2} -${M_PI/2}"/>
   </xacro:monocular_camera>
   <xacro:include filename="$(find mrsl_quadrotor_description)/urdf/dragon_ddk/stereo_camera.urdf.xacro" />
@@ -13,3 +13,22 @@
     <origin xyz="0.1 0.0 0.0" rpy="0 0 0"/>
   </xacro:rgbd_camera>
+  <gazebo reference="imu">
+    <gravity>true</gravity>
+    <sensor name="imu_sensor" type="imu">
+      <always_on>true</always_on>
+      <update_rate>100</update_rate>
+      <visualize>true</visualize>
+      <topic>__default_topic__</topic>
+      <plugin filename="libgazebo_ros_imu_sensor.so" name="imu_plugin">
+        <topicName>imu</topicName>
+        <bodyName>imu_joint</bodyName>
+        <updateRateHZ>100.0</updateRateHZ>
+        <gaussianNoise>0.000</gaussianNoise>
+        <xyzOffset>0 0 0</xyzOffset>
+        <rpyOffset>0 0 0</rpyOffset>
+        <frameName>imu</frameName>
+      </plugin>
+      <pose>0 0 0 0 0 0</pose>
+    </sensor>
+  </gazebo>
 </robot>

File: mrsl_quadrotor_description/urdf/dragon_ddk/stereo_camera.urdf.xacro (robot description, xacro)
@@ -9,5 +9,5 @@
   <xacro:property name="focal_length" value="320" />
   <xacro:property name="hack_baseline" value="0.08" />
-  <xacro:property name="frame_rate" value="15" />
+  <xacro:property name="frame_rate" value="100" />
   <xacro:macro name="stereo_camera" params="name parent *origin">
     <joint name="${name}_joint" type="fixed">
